File: c64modem.sch (KiCad schematic (older format))
At the start: 27 parts, among them CN1 USERPORT, J1 FTDI_PORT, J2 ESP_01, SW1 UP9600, SW2 ESP_RST, SW3 C64_RST, SW4 ESP_PROG, U1 74LVC125, U2 AZ1117-3.3

Commit message: Reroute
Parts:
- removed U1: 74LVC125, Housings_SSOP:TSSOP-14_4.4x5mm_Pitch0.65mm, symbol 74LVC125
- added U1: 74LVC125, Package_SO:TSSOP-14_4.4x5mm_P0.65mm, symbol 74xx:74LVC125
- C1, C2, C4, C5, C7: footprint Capacitors_SMD:C_0603_HandSoldering -> Capacitor_SMD:C_0805_2012Metric_Pad1.15x1.40mm_HandSolder; symbol C -> Device:C
- C3: footprint Capacitors_THT:CP_Radial_D8.0mm_P3.50mm -> Capacitor_THT:CP_Radial_D5.0mm_P2.00mm; symbol CP1 -> Device:CP1
- C6: footprint Capacitors_THT:CP_Radial_D5.0mm_P2.00mm -> Capacitor_THT:CP_Radial_D5.0mm_P2.00mm; symbol CP1 -> Device:CP1
- CN1: symbol USERPORT -> USERPORT:USERPORT
- D1: footprint Diodes_THT:Diode_Bridge_DIP-4_W7.62mm_P5.08mm -> Package_DIP:DIP-4_W7.62mm_LongPads; symbol D_Bridge_+-AA -> c64modem-rescue:D_Bridge_+-AA
- D2, D3, D5: footprint Diodes_THT:D_DO-41_SOD81_P2.54mm_Vertical_AnodeUp -> Diode_THT:D_DO-34_SOD68_P2.54mm_Vertical_AnodeUp; symbol D -> Device:D
- D4: footprint Diodes_SMD:D_SOD-323 -> Diode_SMD:D_SOD-323; symbol D_Schottky -> Device:D_Schottky
- J1: footprint Connectors:PINHEAD1-6 -> Connector_PinHeader_2.54mm:PinHeader_1x06_P2.54mm_Vertical; symbol Conn_01x06 -> c64modem-rescue:Conn_01x06
- J2: footprint Pin_Headers:Pin_Header_Straight_2x04_Pitch2.54mm -> Connector_PinSocket_2.54mm:PinSocket_2x04_P2.54mm_Vertical; symbol Conn_02x04_Odd_Even -> c64modem-rescue:Conn_02x04_Odd_Even
- JP1, JP2: footprint Pin_Headers:Pin_Header_Straight_1x03_Pitch2.54mm -> Connector_PinHeader_2.54mm:PinHeader_1x03_P2.54mm_Vertical; symbol Jumper_NC_Dual -> Device:Jumper_NC_Dual
- R1, R2, R3, R4: footprint Resistors_SMD:R_0603_HandSoldering -> Resistor_SMD:R_0805_2012Metric_Pad1.15x1.40mm_HandSolder; symbol R -> Device:R
- SW1: footprint Buttons_Switches_THT:SW_DIP_x2_W7.62mm_Slide -> Button_Switch_THT:SW_DIP_SPSTx02_Slide_9.78x7.26mm_W7.62mm_P2.54mm; symbol SW_DIP_x02 -> Switch:SW_DIP_x02
- SW2, SW3, SW4: footprint Buttons_Switches_THT:SW_PUSH_6mm -> Button_Switch_THT:SW_PUSH_6mm_H5mm; symbol SW_Push -> c64modem-rescue:SW_Push
- U2: value AZ1117-3.3 -> AMS1117-3.3; footprint TO_SOT_Packages_SMD:SOT-89-3_Handsoldering -> Package_TO_SOT_SMD:SOT-223; symbol AZ1117-3.3 -> Regulator_Linear:AMS1117-3.3
Connections:
- net labels added: ~ESP_RST
- net labels removed: ESP_RST#
- wire segments 112 -> 142
Other:
- note added: "Power to ESP\n"
- moved on the sheet: C2, SW2
