File: c64modem.sch (KiCad schematic (older format))
At the start: 27 parts, among them CN1 USERPORT, J1 FTDI_PORT, SW1 UP9600, SW2 ESP_RST, SW3 C64_RST, SW4 ESP_PROG, U1 74LVC125, U2 AMS1117-3.3

Commit message: Rework.
Parts:
- U2: value AMS1117-3.3 -> LDO1117-3.3; footprint Package_TO_SOT_SMD:SOT-223 -> Package_TO_SOT_SMD:SOT-223-3_TabPin2; symbol Regulator_Linear:AMS1117-3.3 -> Regulator_Linear:LM1117-3.3
Changed lines of the file:
@@
 FTDI_PWR
 $Comp
-L Regulator_Linear:AMS1117-3.3 U2
+L Regulator_Linear:LM1117-3.3 U2
 U 1 1 5ACA5149
 P 5650 5250
 F 0 "U2" H 5500 5375 50  0000 C CNN
-F 1 "AMS1117-3.3" H 5650 5375 50  0000 L CNN
-F 2 "Package_TO_SOT_SMD:SOT-223" H 5650 5500 50  0001 C CIN
+F 1 "LDO1117-3.3" H 5650 5375 50  0000 L CNN
+F 2 "Package_TO_SOT_SMD:SOT-223-3_TabPin2" H 5650 5500 50  0001 C CIN
 F 3 "" H 5650 5250 50  0001 C CNN
 	1    5650 5250
@@
 $EndComp
 $Comp
-L power:VCC #PWR?
+L power:VCC #PWR0102
 U 1 1 5F796975
 P 10300 2300
-F 0 "#PWR?" H 10300 2150 50  0001 C CNN
+F 0 "#PWR0102" H 10300 2150 50  0001 C CNN
 F 1 "VCC" H 10300 2450 50  0000 C CNN
 F 2 "" H 10300 2300 50  0001 C CNN
@@
 $EndComp
 $Comp
-L power:GND #PWR?
+L power:GND #PWR0103
 U 1 1 5F79C0B2
 P 10300 3300
-F 0 "#PWR?" H 10300 3050 50  0001 C CNN
+F 0 "#PWR0103" H 10300 3050 50  0001 C CNN
 F 1 "GND" H 10305 3127 50  0000 C CNN
 F 2 "" H 10300 3300 50  0001 C CNN

Commit message: Rework & add BOM
Parts:
- C3: footprint Capacitor_THT:CP_Radial_D5.0mm_P2.00mm -> Capacitor_THT:CP_Radial_D10.0mm_P5.00mm
Changed lines of the file:
@@
 F 0 "C3" H 4375 5650 50  0000 L CNN
 F 1 "470uF/16V" H 4375 5450 50  0000 L CNN
-F 2 "Capacitor_THT:CP_Radial_D5.0mm_P2.00mm" H 4350 5550 50  0001 C CNN
+F 2 "Capacitor_THT:CP_Radial_D10.0mm_P5.00mm" H 4350 5550 50  0001 C CNN
 F 3 "" H 4350 5550 50  0001 C CNN
 	1    4350 5550
